File: Hardware/graver-controller/driver.kicad_sch (KiCad schematic)
At the start: 0 parts

Commit message: hardware: capture graver controller schematic rev 0.1
Power (LM5164 buck, reverse-polarity P-FET, SS14 ORing, AP2112K),
Driver (UCC27517 + IRLR3410 low side, SS110 + SMBJ24A fast-decay
clamp with SI2309 bypass, 1 ohm shunt, TLV9062 amp and overcurrent
comparator to TIM1_BKIN, GX12 handpiece terminal), MCU (STM32F411CEU6,
25 MHz, USB-C DFU, SWD) and IO (1.3in ST7789 header, EC11E encoder,
NMJ6HCD2 pedal jack). All parts carry LCSC numbers. ERC clean except
one BSS123 library-copy warning.

ADR 0001 folds in the part selection results and deviations: LM5164,
two-Schottky 5 V ORing, BSS123 level shifter, coils >= ~100 ohm,
EC11E15244G1 (30/15), ring-normal plug detect, 1x7 display header,
direct backlight drive, no LSE, PA10 DFU strap, bricks 18-30 V.
Parts:
- added C201: 1uF, Capacitor_SMD:C_0603_1608Metric, symbol Device:C
- added C202, C203, C206, C207: 100nF, Capacitor_SMD:C_0603_1608Metric, symbol Device:C
- added C204: 1nF, Capacitor_SMD:C_0603_1608Metric, symbol Device:C
- added C205: 10nF, Capacitor_SMD:C_0603_1608Metric, symbol Device:C
- added D201: SS110, Diode_SMD:D_SMA, symbol Device:D_Schottky
- added D202: SMBJ24A, Diode_SMD:D_SMB, symbol Device:D_Zener
- added D203: BZT52C12, Diode_SMD:D_SOD-123, symbol Device:D_Zener
- added J201: Handpiece, Connector_Phoenix_MSTB:PhoenixContact_MSTBA_2,5_4-G-5,08_1x04_P5.08mm_Horizontal, symbol Connector:Screw_Terminal_01x04
- added Q201: IRLR3410, Package_TO_SOT_SMD:TO-252-2, symbol Transistor_FET:Q_NMOS_GDS
- added Q202: SI2309CDS, Package_TO_SOT_SMD:SOT-23, symbol Transistor_FET:Q_PMOS_GSD
- added Q203: BSS123, Package_TO_SOT_SMD:SOT-23, symbol Transistor_FET:BSS123
- added R201: 10R, Resistor_SMD:R_0603_1608Metric, symbol Device:R
- added R202, R203, R205, R208: 100k, Resistor_SMD:R_0603_1608Metric, symbol Device:R
- added R204: 1R 1%, Resistor_SMD:R_1206_3216Metric, symbol Device:R
- added R206: 22k, Resistor_SMD:R_0603_1608Metric, symbol Device:R
- added R207: 100R, Resistor_SMD:R_0603_1608Metric, symbol Device:R
- added R209, R211, R213: 1k, Resistor_SMD:R_0603_1608Metric, symbol Device:R
- added R210, R216, R217: 10k, Resistor_SMD:R_0603_1608Metric, symbol Device:R
- added R212: 330R, Resistor_SMD:R_0603_1608Metric, symbol Device:R
- added R214: 1M, Resistor_SMD:R_0603_1608Metric, symbol Device:R
- added R215: 33k, Resistor_SMD:R_0603_1608Metric, symbol Device:R
- added U201: UCC27517DBVR, Package_TO_SOT_SMD:SOT-23-5, symbol Driver_FET:FAN3111C
- added U202: TLV9062IDR, Package_SO:SOIC-8_3.9x4.9mm_P1.27mm, symbol Amplifier_Operational:TLV9062xD
Connections:
- new net +3V3: C203.1, R215.1, R217.1, U202.8 (V+)
- new net +5V: C201.1, C202.1, U201.1 (VDD)
- new net AMP_INN: R210.2, R211.1, U202.2 (-)
- new net AMP_INP: C204.1, R209.2, U202.3 (+)
- new net AMP_OUT: R210.1, R212.1, U202.1
- new net CLAMP: D201.1 (K), D202.1 (K), D203.1 (K), Q202.2 (S), R205.1
- new net CMP_INP: R213.2, R214.2, U202.5 (+)
- new net COIL_NEG: D201.2 (A), J201.2 (Pin_2), Q201.2 (D)
- new net DECAY_SLOW: R207.1
- new net GATE: Q201.1 (G), R201.2, R203.1
- new net GATE_IN: R202.1, U201.3 (IN+)
- new net GND: C201.2, C202.2, C203.2, C204.2, C205.2, C206.2, C207.2, J201.4 (Pin_4), Q203.2 (S), R202.2, R203.2, R204.2, R208.2, R211.2, R216.2, U201.2 (GND), U201.4 (~{IN-}), U202.4 (V-)
- new net I_SENSE: C205.1, R212.2
- new net NTC: C207.1, J201.3 (Pin_3), R217.2
- new net OC_REF: C206.1, R215.2, R216.1, U202.6 (-)
- new net OC_TRIP: R214.1, U202.7
- new net Q202_G: D203.2 (A), Q202.1 (G), R205.2, R206.1
- new net Q203_D: Q203.3 (D), R206.2
- new net Q203_G: Q203.1 (G), R207.2, R208.1
- new net SHUNT_HI: Q201.3 (S), R204.1, R209.1, R213.1
- new net U201_OUT: R201.1, U201.5 (OUT)
- new net VIN: D202.2 (A), J201.1 (Pin_1), Q202.3 (D)
