File: Hardware/graver-controller/driver.kicad_sch (KiCad schematic)
At the start: 33 parts, among them J201 Handpiece, Q201 IRLR3410, Q202 SI2309CDS, Q203 BSS123, U201 UCC27517DBVR, U202 TLV9062IDR

Commit message: hardware: redraw the four schematic sheets with real wiring
The captured sheets connected everything by name with parts scattered on
the page. The sheets are now generated from hand-designed layouts
(Hardware/graver-controller/tools): decoupling caps drawn at their pins,
signal flow left to right, wires inside each block, global labels only
where a net crosses sheets. Power is two rows, MCU and IO fit A4.

Circuit unchanged: verify.sh compares the XML netlist against the
captured sheets kept in tools/ref (117 components with values,
footprints and LCSC fields, 65 nets by pin set) - identical. ERC: 0
violations. Q203 uses the generic Q_NMOS_GSD symbol (value BSS123),
which removes the library-mismatch warning.
Parts:
- removed Q203: BSS123, Package_TO_SOT_SMD:SOT-23, symbol Transistor_FET:BSS123
- added Q203: BSS123, Package_TO_SOT_SMD:SOT-23, symbol Transistor_FET:Q_NMOS_GSD
Connections:
- net GND: now also Q203.2 (S)
- net AMP_INN: no longer names the net of R210.2, R211.1, U202.2 (-)
- net AMP_INP: no longer names the net of C204.1, R209.2, U202.3 (+)
- net AMP_OUT: no longer names the net of R210.1, R212.1, U202.1
- net CMP_INP: no longer names the net of R213.2, R214.2, U202.5 (+)
- net GATE: no longer names the net of Q201.1 (G), R201.2, R203.1
- net Q202_G: no longer names the net of D203.2 (A), Q202.1 (G), R205.2, R206.1
- net Q203_D: no longer names the net of R206.2
- net Q203_D: now also Q203.3 (D)
- net Q203_G: no longer names the net of R207.2, R208.1
- net Q203_G: now also Q203.1 (G)
- net U201_OUT: no longer names the net of R201.1, U201.5 (OUT)
Other:
- note added: "0.26 A -> 2.9 V at the ADC"
- note added: "DECAY_SLOW high: Q202 shorts D202, plain diode flyback"
- note added: "R204: Kelvin-route to R209/R213"
- note added: "fast decay: coil sees VIN + 24 V TVS at turn-off"
- note added: "optional NTC"
- note added: "trip ~0.77 A, 1M hysteresis"
