File: Hardware/graver-controller/driver.kicad_sch (KiCad schematic)
At the start: 33 parts, among them J201 Handpiece, Q201 IRLR3410, Q202 SI2309CDS, Q203 BSS123, U201 UCC27517DBVR, U202 TLV9062IDR

Commit message: hardware: wire pads instead of connectors, board to 95 x 70
ADR 0003 Decision 9. Every board connector except USB-C becomes a row of
plated through-holes and the rotary encoder moves off the board onto wires;
Jan solders the looms at box build. The mating halves were the sourcing
problem, not the board halves, and the four connectors dropped here were
also the four parts whose footprints were still unverified against real
hardware.

Schematic (ERC 0, netlist diffed pad-by-pad - every difference was an
auto-generated net NAME following its anchor pin, no connectivity changed):

- J101 Barrel_Jack_Switch -> Conn_01x02, SolderWire-1sqmm 1x02, 1.4 mm
- J201 -> PinHeader_1x04, J401 -> PinHeader_1x07
- J402 AudioJack3_SwitchTR -> Conn_01x04 (TIP, RN, RING, SLV)
- SW401 RotaryEncoder_Switch_MP -> J403 Conn_01x04 (A, GND, B, SW)
- the five pad rows carry no LCSC/MPN: they are holes, not parts, and an
  empty field reads as a schematic-parity mismatch
- three orphaned no-connect flags removed with the old unused pins

Board 110 x 70 -> 95 x 70: measured on the routed board, everything except
the connectors, the encoder and the mounting holes fits in 84.5 x 64.0 mm,
so the connectors were setting the width. 95 also brings the long side
under JLC's 100 x 100 price band.

State: 0 DRC errors, 0 schematic parity, 3 unconnected pad pairs (+5V and
two GND, all short same-net gaps), 11 warnings, 126 vias, all placement
checks and ADR criteria PASS, all eight per-net width floors PASS.

Tooling:

- outline 95 x 70 in place.py, copper.py, silk.py and render.sh
- rear pad rows inset from the edge (negative overhang): J101's 2.7 mm pads
  sitting flush broke the 0.3 mm copper-to-edge rule
- silk legends rewritten; the two MIDDLE pads of each 1x4 rear row had no
  sideways escape at 2.54 mm pitch and silently got no label, which on the
  handpiece row is 24 V versus the NTC input. Pin numbers dropped and the
  seed pushed to 3.6 mm; 24 of 24 legends now place on seed.
- copper.py BRIDGE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
Parts:
- J201: value Handpiece -> Handpiece pads 1x4; footprint Connector_Phoenix_MSTB:PhoenixContact_MSTBA_2,5_4-G-5,08_1x04_P5.08mm_Horizontal -> Connector_PinHeader_2.54mm:PinHeader_1x04_P2.54mm_Vertical; LCSC C8446 -> (none); MPN WJ2EDGRC-5.08-4P -> (none)
Changed lines of the file:
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@@
 			)
 		)
-		(property "Value" "Handpiece"
+		(property "Value" "Handpiece pads 1x4"
 			(at 154.94 53.34 270)
 			(show_name no)
@@
 			)
 		)
-		(property "Footprint" "Connector_Phoenix_MSTB:PhoenixContact_MSTBA_2,5_4-G-5,08_1x04_P5.08mm_Horizontal"
+		(property "Footprint" "Connector_PinHeader_2.54mm:PinHeader_1x04_P2.54mm_Vertical"
 			(at 163.83 60.96 0)
 			(hide yes)
@@
 			(at 163.83 60.96 0)
 			(hide yes)
-			(show_name no)
-			(do_not_autoplace no)
-			(effects
-				(font
-					(size 1.27 1.27)
-				)
-			)
-		)
-		(property "LCSC" "C8446"
-			(at 163.83 60.96 0)
-			(hide yes)
-			(show_name no)
-			(do_not_autoplace no)
-			(effects
-				(font
-					(size 1.27 1.27)
-				)
-			)
-		)
-		(property "MPN" "WJ2EDGRC-5.08-4P"
-			(at 163.83 60.96 0)
-			(hide yes)
