File: Hardware/graver-controller/mcu.kicad_sch (KiCad schematic)
At the start: 0 parts

Commit message: hardware: capture graver controller schematic rev 0.1
Power (LM5164 buck, reverse-polarity P-FET, SS14 ORing, AP2112K),
Driver (UCC27517 + IRLR3410 low side, SS110 + SMBJ24A fast-decay
clamp with SI2309 bypass, 1 ohm shunt, TLV9062 amp and overcurrent
comparator to TIM1_BKIN, GX12 handpiece terminal), MCU (STM32F411CEU6,
25 MHz, USB-C DFU, SWD) and IO (1.3in ST7789 header, EC11E encoder,
NMJ6HCD2 pedal jack). All parts carry LCSC numbers. ERC clean except
one BSS123 library-copy warning.

ADR 0001 folds in the part selection results and deviations: LM5164,
two-Schottky 5 V ORing, BSS123 level shifter, coils >= ~100 ohm,
EC11E15244G1 (30/15), ring-normal plug detect, 1x7 display header,
direct backlight drive, no LSE, PA10 DFU strap, bricks 18-30 V.
Parts:
- added C301, C302, C303, C304, C309: 100nF, Capacitor_SMD:C_0603_1608Metric, symbol Device:C
- added C305, C308: 4.7uF, Capacitor_SMD:C_0603_1608Metric, symbol Device:C
- added C306: 1uF, Capacitor_SMD:C_0603_1608Metric, symbol Device:C
- added C307: 10nF, Capacitor_SMD:C_0603_1608Metric, symbol Device:C
- added C310, C311: 12pF C0G, Capacitor_SMD:C_0402_1005Metric, symbol Device:C
- added D301: STAT red, LED_SMD:LED_0603_1608Metric, symbol Device:LED
- added FB301: 600R@100MHz, Inductor_SMD:L_0603_1608Metric, symbol Device:FerriteBead_Small
- added J301: USB-C, Connector_USB:USB_C_Receptacle_HRO_TYPE-C-31-M-12, symbol Connector:USB_C_Receptacle_USB2.0_16P
- added J302: SWD, Connector_PinHeader_2.54mm:PinHeader_1x05_P2.54mm_Vertical, symbol Connector_Generic:Conn_01x05
- added R301, R303, R307: 10k, Resistor_SMD:R_0603_1608Metric, symbol Device:R
- added R302, R304: 1k, Resistor_SMD:R_0603_1608Metric, symbol Device:R
- added R305, R306: 5.1k, Resistor_SMD:R_0603_1608Metric, symbol Device:R
- added SW301: BOOT0, Button_Switch_SMD:SW_Push_1P1T_XKB_TS-1187A, symbol Switch:SW_Push
- added SW302: RESET, Button_Switch_SMD:SW_Push_1P1T_XKB_TS-1187A, symbol Switch:SW_Push
- added U301: STM32F411CEU6, Package_DFN_QFN:QFN-48-1EP_7x7mm_P0.5mm_EP5.6x5.6mm, symbol MCU_ST_STM32F4:STM32F411CEUx
- added U302: USBLC6-2SC6, Package_TO_SOT_SMD:SOT-23-6, symbol Power_Protection:USBLC6-2SC6
- added Y301: 25MHz 10pF, Crystal:Crystal_SMD_3225-4Pin_3.2x2.5mm, symbol Device:Crystal_GND24
Connections:
- new net +3V3: C301.1, C302.1, C303.1, C304.1, C305.1, FB301.1, J302.1 (Pin_1), R304.1, R307.2, SW301.2, U301.1 (VBAT), U301.24 (VDD), U301.36 (VDD), U301.48 (VDD)
- new net BOOT0: R301.1, R302.1, U301.44 (BOOT0)
- new net BOOT0_SW: R302.2, SW301.1
- new net BOOT1: R303.1, U301.20 (PB2)
- new net DECAY_SLOW: U301.27 (PB14)
- new net ENC_A: U301.40 (PB4)
- new net ENC_B: U301.41 (PB5)
- new net ENC_SW: U301.43 (PB7)
- new net GATE_IN: U301.29 (PA8)
- new net GND: C301.2, C302.2, C303.2, C304.2, C305.2, C306.2, C307.2, C308.2, C309.2, C310.2, C311.2, J301.A1 (GND), J301.A12 (GND), J301.B1 (GND), J301.B12 (GND), J301.SH (SHIELD), J302.5 (Pin_5), R301.2, R303.2, R305.2, R306.2, SW302.2, U301.23 (VSS), U301.35 (VSS), U301.47 (VSS), U301.49 (VSS), U301.8 (VSSA), U302.2 (GND), Y301.2 (G), Y301.4 (G)
- new net I_SENSE: U301.16 (PA6)
- new net LCD_BL: U301.42 (PB6)
- new net LCD_DC: U301.21 (PB10)
- new net LCD_MOSI: U301.17 (PA7)
- new net LCD_RST: U301.28 (PB15)
- new net LCD_SCK: U301.15 (PA5)
- new net LED_STAT: D301.1 (K), U301.2 (PC13)
- new net MCU_VCAP: C308.1, U301.22 (VCAP1)
- new net NRST: C309.1, J302.4 (Pin_4), SW302.1, U301.7 (NRST)
- new net NTC: U301.19 (PB1)
- new net OC_TRIP: U301.25 (PB12)
- new net OSC_IN: C310.1, U301.5 (PH0), Y301.1
- new net OSC_OUT: C311.1, U301.6 (PH1), Y301.3
- new net PA10_PU: R307.1, U301.31 (PA10)
- new net PEDAL_RING: U301.12 (PA2)
- new net PEDAL_TIP: U301.11 (PA1)
- new net STAT_LED_A: D301.2 (A), R304.2
- new net SWCLK: J302.3 (Pin_3), U301.37 (PA14)
- new net SWDIO: J302.2 (Pin_2), U301.34 (PA13)
- new net USB_CC1: J301.A5 (CC1), R305.1
- new net USB_CC2: J301.B5 (CC2), R306.1
- new net USB_DM: J301.A7 (D-), J301.B7 (D-), U301.32 (PA11), U302.1 (I/O1), U302.6 (I/O1)
- new net USB_DP: J301.A6 (D+), J301.B6 (D+), U301.33 (PA12), U302.3 (I/O2), U302.4 (I/O2)
- new net VBUS: J301.A4 (VBUS), J301.A9 (VBUS), J301.B4 (VBUS), J301.B9 (VBUS), U302.5 (VBUS)
- new net VDDA: C306.1, C307.1, FB301.2, U301.9 (VDDA)
- new net VIN_SENSE: U301.18 (PB0)
- no-connect marks 0 -> 13
