File: Hardware/graver-controller/mcu.kicad_sch (KiCad schematic)
At the start: 27 parts, among them J301 USB-C, J302 SWD, SW301 BOOT0, SW302 RESET, U301 STM32F411CEU6, U302 USBLC6-2SC6, Y301 25MHz 10pF

Commit message: hardware: redraw the four schematic sheets with real wiring
The captured sheets connected everything by name with parts scattered on
the page. The sheets are now generated from hand-designed layouts
(Hardware/graver-controller/tools): decoupling caps drawn at their pins,
signal flow left to right, wires inside each block, global labels only
where a net crosses sheets. Power is two rows, MCU and IO fit A4.

Circuit unchanged: verify.sh compares the XML netlist against the
captured sheets kept in tools/ref (117 components with values,
footprints and LCSC fields, 65 nets by pin set) - identical. ERC: 0
violations. Q203 uses the generic Q_NMOS_GSD symbol (value BSS123),
which removes the library-mismatch warning.
Connections:
- net BOOT0: no longer names the net of R301.1, R302.1, U301.44 (BOOT0)
- net BOOT0_SW: no longer names the net of R302.2, SW301.1
- net BOOT1: no longer names the net of R303.1, U301.20 (PB2)
- net MCU_VCAP: no longer names the net of C308.1, U301.22 (VCAP1)
- net PA10_PU: no longer names the net of R307.1, U301.31 (PA10)
- net STAT_LED_A: no longer names the net of D301.2 (A), R304.2
Other:
- note added: "C301-C304: one per VDD/VBAT pin, C305 bulk"
- note added: "hold at power-up: USB DFU"
