File: Hardware/graver-controller/power.kicad_sch (KiCad schematic)
At the start: 0 parts

Commit message: hardware: capture graver controller schematic rev 0.1
Power (LM5164 buck, reverse-polarity P-FET, SS14 ORing, AP2112K),
Driver (UCC27517 + IRLR3410 low side, SS110 + SMBJ24A fast-decay
clamp with SI2309 bypass, 1 ohm shunt, TLV9062 amp and overcurrent
comparator to TIM1_BKIN, GX12 handpiece terminal), MCU (STM32F411CEU6,
25 MHz, USB-C DFU, SWD) and IO (1.3in ST7789 header, EC11E encoder,
NMJ6HCD2 pedal jack). All parts carry LCSC numbers. ERC clean except
one BSS123 library-copy warning.

ADR 0001 folds in the part selection results and deviations: LM5164,
two-Schottky 5 V ORing, BSS123 level shifter, coils >= ~100 ohm,
EC11E15244G1 (30/15), ring-normal plug detect, 1x7 display header,
direct backlight drive, no LSE, PA10 DFU strap, bricks 18-30 V.
Parts:
- added C101: 470uF 63V, Capacitor_THT:CP_Radial_D12.5mm_P5.00mm, symbol Device:C_Polarized
- added C102: 1uF 100V, Capacitor_SMD:C_0805_2012Metric, symbol Device:C
- added C103, C107: 100nF 100V, Capacitor_SMD:C_0805_2012Metric, symbol Device:C
- added C104: 100nF, Capacitor_SMD:C_0603_1608Metric, symbol Device:C
- added C105, C106: 2.2uF 100V, Capacitor_SMD:C_1206_3216Metric, symbol Device:C
- added C108: 2.2nF 50V, Capacitor_SMD:C_0603_1608Metric, symbol Device:C
- added C109: 3.3nF, Capacitor_SMD:C_0603_1608Metric, symbol Device:C
- added C110: 100pF C0G, Capacitor_SMD:C_0603_1608Metric, symbol Device:C
- added C111, C112: 22uF 25V, Capacitor_SMD:C_0805_2012Metric, symbol Device:C
- added C113, C114: 1uF, Capacitor_SMD:C_0603_1608Metric, symbol Device:C
- added C115: 10uF, Capacitor_SMD:C_0805_2012Metric, symbol Device:C
- added D101: BZT52C12, Diode_SMD:D_SOD-123, symbol Device:D_Zener
- added D102: SMBJ36A, Diode_SMD:D_SMB, symbol Device:D_Zener
- added D103, D105: SS14, Diode_SMD:D_SMA, symbol Device:D_Schottky
- added D104: PWR green, LED_SMD:LED_0805_2012Metric, symbol Device:LED
- added F101: 1A slow, Fuse:Fuse_1206_3216Metric, symbol Device:Fuse
- added J101: DC jack 5.5x2.1, Connector_BarrelJack:BarrelJack_Horizontal, symbol Connector:Barrel_Jack_Switch
- added L101: 33uH, Inductor_SMD:L_Changjiang_FXL0630, symbol Device:L
- added Q101: DMP6023LE, Package_TO_SOT_SMD:SOT-223-3_TabPin2, symbol Transistor_FET:Q_PMOS_GDS
- added R101, R102: 100k, Resistor_SMD:R_0603_1608Metric, symbol Device:R
- added R103: 8.2k, Resistor_SMD:R_0603_1608Metric, symbol Device:R
- added R104: 2.2k, Resistor_SMD:R_0603_1608Metric, symbol Device:R
- added R105: 1M, Resistor_SMD:R_0603_1608Metric, symbol Device:R
- added R106: 120k, Resistor_SMD:R_0603_1608Metric, symbol Device:R
- added R107: 33k 1%, Resistor_SMD:R_0603_1608Metric, symbol Device:R
- added R108: 150k, Resistor_SMD:R_0603_1608Metric, symbol Device:R
- added R109: 340k 1%, Resistor_SMD:R_0603_1608Metric, symbol Device:R
- added R110: 100k 1%, Resistor_SMD:R_0603_1608Metric, symbol Device:R
- added U101: LM5164DDAR, Package_SO:HSOP-8-1EP_3.9x4.9mm_P1.27mm_EP2.41x3.1mm_ThermalVias, symbol Regulator_Switching:LM5164DDA
- added U102: AP2112K-3.3, Package_TO_SOT_SMD:SOT-23-5, symbol Regulator_Linear:AP2112K-3.3
Connections:
- new net +3V3: C114.1, C115.1, R104.1, U102.5 (VOUT)
- new net +5V: C113.1, D103.1 (K), D105.1 (K), U102.1 (VIN), U102.3 (EN)
- new net BUCK_5V: C109.2, C111.1, C112.1, D105.2 (A), L101.2, R109.1
- new net BUCK_BST: C108.1, U101.7 (BST)
- new net BUCK_EN: R105.2, R106.1, U101.3 (EN/UVLO)
- new net BUCK_FB: C110.2, R109.2, R110.1, U101.5 (FB)
- new net BUCK_RIPPLE: C109.1, C110.1, R108.2
- new net BUCK_RON: R107.1, U101.4 (RON)
- new net BUCK_SW: C108.2, L101.1, R108.1, U101.8 (SW)
- new net GND: C101.2, C102.2, C103.2, C104.2, C105.2, C106.2, C107.2, C111.2, C112.2, C113.2, C114.2, C115.2, D102.2 (A), D104.1 (K), J101.2, R101.2, R103.2, R106.2, R107.2, R110.2, U101.1 (GND), U101.9 (EP), U102.2 (GND)
- new net PWR_LED_A: D104.2 (A), R104.2
- new net Q101_G: D101.2 (A), Q101.1 (G), R101.1
- new net VBUS: D103.2 (A)
- new net VIN: C101.1, C102.1, C103.1, C105.1, C106.1, C107.1, D101.1 (K), D102.1 (K), Q101.3 (S), R102.1, R105.1, U101.2 (VIN)
- new net VIN_F: F101.2, Q101.2 (D)
- new net VIN_RAW: F101.1, J101.1
- new net VIN_SENSE: C104.1, R102.2, R103.1
- no-connect marks 0 -> 3
