File: Hardware/graver-controller/io.kicad_sch (KiCad schematic)
At the start: 21 parts, among them J401 LCD 1x7, J402 NMJ6HCD2, SW401 EC11E15244G1, U401 PESD5V0S2BT

Commit message: hardware: retire the schematic generator, J401 becomes a JST XH header
eeschema is the source of truth from here (ADR 0003). build.py refuses to
overwrite the sheets without --force-overwrite, verify.sh keeps ERC and
the renders and now fails on ERC violations. J401 (display): B7B-XH-A,
C144398, 2.50 mm pitch footprint; nets and pin order unchanged, ERC 0.
Parts:
- J401: value LCD 1x7 -> LCD XH 1x7; footprint Connector_PinSocket_2.54mm:PinSocket_1x07_P2.54mm_Vertical -> Connector_JST:JST_XH_B7B-XH-A_1x07_P2.50mm_Vertical; LCSC C2832270 -> C144398; MPN PM254V-11-07-H85 -> B7B-XH-A(LF)(SN)
Changed lines of the file:
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@@
 			)
 		)
-		(property "Value" "LCD 1x7"
+		(property "Value" "LCD XH 1x7"
 			(at 71.12 74.93 0)
 			(show_name no)
@@
 			)
 		)
-		(property "Footprint" "Connector_PinSocket_2.54mm:PinSocket_1x07_P2.54mm_Vertical"
+		(property "Footprint" "Connector_JST:JST_XH_B7B-XH-A_1x07_P2.50mm_Vertical"
 			(at 73.66 63.5 0)
 			(hide yes)
@@
 			)
 		)
-		(property "LCSC" "C2832270"
+		(property "LCSC" "C144398"
 			(at 73.66 63.5 0)
 			(hide yes)
@@
 			)
 		)
-		(property "MPN" "PM254V-11-07-H85"
+		(property "MPN" "B7B-XH-A(LF)(SN)"
 			(at 73.66 63.5 0)
 			(hide yes)

Commit message: hardware: wire pads instead of connectors, board to 95 x 70
ADR 0003 Decision 9. Every board connector except USB-C becomes a row of
plated through-holes and the rotary encoder moves off the board onto wires;
Jan solders the looms at box build. The mating halves were the sourcing
problem, not the board halves, and the four connectors dropped here were
also the four parts whose footprints were still unverified against real
hardware.

Schematic (ERC 0, netlist diffed pad-by-pad - every difference was an
auto-generated net NAME following its anchor pin, no connectivity changed):

- J101 Barrel_Jack_Switch -> Conn_01x02, SolderWire-1sqmm 1x02, 1.4 mm
- J201 -> PinHeader_1x04, J401 -> PinHeader_1x07
- J402 AudioJack3_SwitchTR -> Conn_01x04 (TIP, RN, RING, SLV)
- SW401 RotaryEncoder_Switch_MP -> J403 Conn_01x04 (A, GND, B, SW)
- the five pad rows carry no LCSC/MPN: they are holes, not parts, and an
  empty field reads as a schematic-parity mismatch
- three orphaned no-connect flags removed with the old unused pins

Board 110 x 70 -> 95 x 70: measured on the routed board, everything except
the connectors, the encoder and the mounting holes fits in 84.5 x 64.0 mm,
so the connectors were setting the width. 95 also brings the long side
under JLC's 100 x 100 price band.

State: 0 DRC errors, 0 schematic parity, 3 unconnected pad pairs (+5V and
two GND, all short same-net gaps), 11 warnings, 126 vias, all placement
checks and ADR criteria PASS, all eight per-net width floors PASS.

Tooling:

- outline 95 x 70 in place.py, copper.py, silk.py and render.sh
- rear pad rows inset from the edge (negative overhang): J101's 2.7 mm pads
  sitting flush broke the 0.3 mm copper-to-edge rule
- silk legends rewritten; the two MIDDLE pads of each 1x4 rear row had no
  sideways escape at 2.54 mm pitch and silently got no label, which on the
  handpiece row is 24 V versus the NTC input. Pin numbers dropped and the
  seed pushed to 3.6 mm; 24 of 24 legends now place on seed.
- copper.py BRIDGE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
Parts:
- removed J402: NMJ6HCD2, Connector_Audio:Jack_6.35mm_Neutrik_NMJ6HCD2_Horizontal, symbol Connector_Audio:AudioJack3_SwitchTR
- removed SW401: EC11E15244G1, Rotary_Encoder:RotaryEncoder_Alps_EC11E-Switch_Vertical_H20mm, symbol Device:RotaryEncoder_Switch_MP
- added J402: Pedal pads 1x4, Connector_PinHeader_2.54mm:PinHeader_1x04_P2.54mm_Vertical, symbol Connector_Generic:Conn_01x04
- added J403: Encoder pads 1x4, Connector_PinHeader_2.54mm:PinHeader_1x04_P2.54mm_Vertical, symbol Connector_Generic:Conn_01x04
- J401: value LCD XH 1x7 -> LCD pads 1x7; footprint Connector_JST:JST_XH_B7B-XH-A_1x07_P2.50mm_Vertical -> Connector_PinHeader_2.54mm:PinHeader_1x07_P2.54mm_Vertical; LCSC C144398 -> (none); MPN B7B-XH-A(LF)(SN) -> (none)
Connections:
- net ENC_A: now also J403.1 (Pin_1)
- net ENC_B: now also J403.3 (Pin_3)
- net ENC_SW: now also J403.4 (Pin_4)
- net GND: now also J402.2 (Pin_2), J402.4 (Pin_4), J403.2 (Pin_2)
- net at R405.2, R406.1, U401.2 (A2): now also J402.3 (Pin_3)
- net at R407.2, R408.1, U401.1 (A1): now also J402.1 (Pin_1)
- no-connect marks 2 -> 0
Other:
- note added: "EC11E15244G1 or any EC11: 30 detents / 15 pulses, TIM3 encoder mode"
- note added: "Encoder is OFF-BOARD, in the cover plate: 4 wires to J403"
- note added: "Pedal socket is OFF-BOARD: tip = wiper, ring = 3V3 feed, sleeve = GND"
- note added: "no plug or mono plug: RN grounds the ring -> firmware sees no pedal (needs a TRS socket)"
- note removed: "EC11E15244G1: 30 detents / 15 pulses, TIM3 encoder mode"
- note removed: "TRS: tip = wiper, ring = 3V3 feed, sleeve = GND"
- note removed: "no plug or mono plug: RN grounds the ring -> firmware sees no pedal"
Changed lines of the file:
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@@
 		(title "IO")
 	)
-	(text "no plug or mono plug: RN grounds the ring -> firmware sees no pedal"
+	(text "no plug or mono plug: RN grounds the ring -> firmware sees no pedal (needs a TRS socket)"
 		(exclude_from_sim no)
 		(at 58.42 157.48 0)
@@
 		)
 	)
-	(text "EC11E15244G1: 30 detents / 15 pulses, TIM3 encoder mode"
+	(text "Encoder is OFF-BOARD, in the cover plate: 4 wires to J403"
 		(exclude_from_sim no)
 		(at 109.22 92.71 0)
@@
 		)
 	)
+	(text "EC11E15244G1 or any EC11: 30 detents / 15 pulses, TIM3 encoder mode"
+		(exclude_from_sim no)
+		(at 109.22 95.25 0)
+		(effects
+			(font
+				(size 1.27 1.27)
+			)
+			(justify left top)
+		)
+	)
 	(text "1.3in ST7789 240x240 module, 3V3, no CS: SPI mode 3"
 		(exclude_from_sim no)
@@
 		)
 	)
-	(text "TRS: tip = wiper, ring = 3V3 feed, sleeve = GND"
+	(text "Pedal socket is OFF-BOARD: tip = wiper, ring = 3V3 feed, sleeve = GND"
 		(exclude_from_sim no)
 		(at 58.42 154.94 0)
@@
 		(color 0 0 0 0)
 	)
-	(no_connect
-		(at 152.4 71.12)
-	)
-	(no_connect
-		(at 78.74 132.08)
-	)
 	(wire
 		(pts
@@
 	(wire
 		(pts
-			(xy 160.02 66.04) (xy 165.1 66.04)
-		)
-		(stroke
-			(width 0)
-			(type default)
-		)
-	)
-	(wire
-		(pts
 			(xy 63.5 71.12) (xy 63.5 76.2)
 		)
@@
 	)
 	(symbol
-		(lib_id "Connector_Audio:AudioJack3_SwitchTR")
-		(at 73.66 124.46 0)
+		(lib_id "Connector_Generic:Conn_01x04")
+		(at 73.66 127.0 180)
 		(unit 1)
 		(body_style 1)
@@
 		(dnp no)
 		(property "Reference" "J402"
-			(at 63.5 114.3 0)
+			(at 71.11999999999999 116.84 0)
 			(show_name no)
 			(do_not_autoplace no)
@@
 			)
 		)
-		(property "Value" "NMJ6HCD2"
-			(at 63.5 137.16 0)
+		(property "Value" "Pedal pads 1x4"
+			(at 71.11999999999999 137.16 0)
 			(show_name no)
 			(do_not_autoplace no)
@@
 			)
 		)
-		(property "Footprint" "Connector_Audio:Jack_6.35mm_Neutrik_NMJ6HCD2_Horizontal"
-			(at 73.66 124.46 0)
+		(property "Footprint" "Connector_PinHeader_2.54mm:PinHeader_1x04_P2.54mm_Vertical"
+			(at 73.66 127.0 0)
 			(hide yes)
 			(show_name no)
@@
 		)
 		(property "Datasheet" ""
-			(at 73.66 124.46 0)
+			(at 73.66 127.0 0)
 			(hide yes)
 			(show_name no)
@@
 		)
 		(property "Description" ""
-			(at 73.66 124.46 0)
-			(hide yes)
-			(show_name no)
-			(do_not_autoplace no)
-			(effects
-				(font
-					(size 1.27 1.27)
-				)
-			)
-		)
-		(property "LCSC" "C368502"
-			(at 73.66 124.46 0)
-			(hide yes)
-			(show_name no)
-			(do_not_autoplace no)
-			(effects
-				(font
-					(size 1.27 1.27)
-				)
-			)
-		)
-		(property "MPN" "NMJ6HCD2"
-			(at 73.66 124.46 0)
+			(at 73.66 127.0 0)
 			(hide yes)
 			(show_name no)
@@
 			)
 		)
-		(pin "R"
-		)
-		(pin "RN"
+		(pin "1"
 		)
-		(pin "S"
+		(pin "2"
 		)
-		(pin "T"
+		(pin "3"
 		)
-		(pin "TN"
+		(pin "4"
 		)
 		(instances
@@
 			)
 		)
-		(property "Value" "LCD XH 1x7"
+		(property "Value" "LCD pads 1x7"
 			(at 71.12 74.93 0)
 			(show_name no)
@@
 			)
 		)
-		(property "Footprint" "Connector_JST:JST_XH_B7B-XH-A_1x07_P2.50mm_Vertical"
+		(property "Footprint" "Connector_PinHeader_2.54mm:PinHeader_1x07_P2.54mm_Vertical"
 			(at 73.66 63.5 0)
 			(hide yes)
@@
 			)
 		)
-		(property "LCSC" "C144398"
-			(at 73.66 63.5 0)
-			(hide yes)
-			(show_name no)
-			(do_not_autoplace no)
-			(effects
-				(font
-					(size 1.27 1.27)
-				)
-			)
-		)
-		(property "MPN" "B7B-XH-A(LF)(SN)"
-			(at 73.66 63.5 0)
-			(hide yes)
-			(show_name no)
-			(do_not_autoplace no)
-			(effects
-				(font
-					(size 1.27 1.27)
-				)
-			)
-		)
 		(pin "1"
 		)
@@
 	)
 	(symbol
-		(lib_id "power:GND")
-		(at 165.1 66.04 0)
-		(unit 1)
-		(body_style 1)
-		(exclude_from_sim no)
-		(in_bom yes)
-		(on_board yes)
-		(in_pos_files yes)
-		(dnp no)
-		(property "Reference" "#PWR410"
-			(at 165.1 72.39 0)
-			(hide yes)
-			(show_name no)
-			(do_not_autoplace no)
-			(effects
-				(font
-					(size 1.27 1.27)
-				)
-			)
-		)
-		(property "Value" "GND"
-			(at 165.1 71.12 0)
-			(show_name no)
-			(do_not_autoplace no)
-			(effects
-				(font
-					(size 1.27 1.27)
-				)
-			)
-		)
-		(property "Footprint" ""
-			(at 165.1 66.04 0)
-			(hide yes)
-			(show_name no)
-			(do_not_autoplace no)
-			(effects
-				(font
-					(size 1.27 1.27)
-				)
-			)
-		)
-		(property "Datasheet" ""
-			(at 165.1 66.04 0)
-			(hide yes)
-			(show_name no)
-			(do_not_autoplace no)
-			(effects
-				(font
-					(size 1.27 1.27)
-				)
-			)
-		)
-		(property "Description" ""
-			(at 165.1 66.04 0)
-			(hide yes)
-			(show_name no)
-			(do_not_autoplace no)
-			(effects
-				(font
-					(size 1.27 1.27)
-				)
-			)
-		)
-		(pin "1"
-		)
-		(instances
-			(project "graver-controller"
-				(path "/d303ff23-e0bc-456d-81fe-4c8aea3d493e/2f15ba9a-6165-4167-85f8-f67e3d99cc62"
-					(reference "#PWR410")
-					(unit 1)
-				)
-			)
-		)
-	)
-	(symbol
 		(lib_id "Device:R")
 		(at 58.42 76.2 90)
@@
 	)
 	(symbol
-		(lib_id "Device:RotaryEncoder_Switch_MP")
-		(at 152.4 63.5 0)
+		(lib_id "Connector_Generic:Conn_01x04")
+		(at 149.86 63.5 0)
 		(unit 1)
 		(body_style 1)
@@
 		(in_pos_files yes)
 		(dnp no)
-		(property "Reference" "SW401"
-			(at 147.32 53.34 0)
+		(property "Reference" "J403"
+			(at 147.32000000000002 53.34 0)
 			(show_name no)
 			(do_not_autoplace no)
@@
 			)
 		)
-		(property "Value" "EC11E15244G1"
-			(at 157.48 77.47 0)
+		(property "Value" "Encoder pads 1x4"
+			(at 158.75 73.66 0)
 			(show_name no)
 			(do_not_autoplace no)
@@
 			)
 		)
-		(property "Footprint" "Rotary_Encoder:RotaryEncoder_Alps_EC11E-Switch_Vertical_H20mm"
-			(at 152.4 63.5 0)
+		(property "Footprint" "Connector_PinHeader_2.54mm:PinHeader_1x04_P2.54mm_Vertical"
+			(at 149.86 63.5 0)
 			(hide yes)
 			(show_name no)
@@
 		)
 		(property "Datasheet" ""
-			(at 152.4 63.5 0)
+			(at 149.86 63.5 0)
 			(hide yes)
 			(show_name no)
@@
 		)
 		(property "Description" ""
-			(at 152.4 63.5 0)
-			(hide yes)
-			(show_name no)
-			(do_not_autoplace no)
-			(effects
-				(font
-					(size 1.27 1.27)
-				)
-			)
-		)
-		(property "LCSC" "C370970"
-			(at 152.4 63.5 0)
-			(hide yes)
-			(show_name no)
-			(do_not_autoplace no)
-			(effects
-				(font
-					(size 1.27 1.27)
-				)
-			)
-		)
-		(property "MPN" "EC11E15244G1"
-			(at 152.4 63.5 0)
+			(at 149.86 63.5 0)
 			(hide yes)
 			(show_name no)
@@
 			)
 		)
-		(pin "A"
-		)
-		(pin "B"
-		)
-		(pin "C"
+		(pin "1"
 		)
-		(pin "MP"
+		(pin "2"
 		)
-		(pin "S1"
+		(pin "3"
 		)
-		(pin "S2"
+		(pin "4"
 		)
 		(instances
 			(project "graver-controller"
 				(path "/d303ff23-e0bc-456d-81fe-4c8aea3d493e/2f15ba9a-6165-4167-85f8-f67e3d99cc62"
-					(reference "SW401")
+					(reference "J403")
 					(unit 1)
 				)
@@
 		)
 	)
+	(wire
+		(pts
+			(xy 144.78 68.58) (xy 144.78 71.12)
+		)
+		(stroke
+			(width 0)
+			(type default)
+		)
+	)
+	(wire
+		(pts
+			(xy 144.78 71.12) (xy 160.02 71.12)
+		)
+		(stroke
+			(width 0)
+			(type default)
+		)
+	)
+	(wire
+		(pts
+			(xy 160.02 71.12) (xy 160.02 60.96)
+		)
+		(stroke
+			(width 0)
+			(type default)
+		)
+	)
